Commit message: Fix swarm mapping: stateless merge, shared world frame, stable rover
- map_merge_node: keep only the latest map per robot and rebuild
  /map_merged from scratch on a 1 s sim-time timer, published in
  'world'. The old grid accumulated every stale wall forever. Use
  floor() instead of int() for output cell indices.
- slam_swarm.launch.py: static world -> <name>/map transforms from
  fleet_config, so every robot's TF tree hangs off one root.
- rover.urdf.xacro: move the chassis 3 cm (scout) / 6 cm (mapper)
  ahead of the axle. The rovers were tipping onto their tails
  (measured 15.2 / 12.9 deg) and the tilted lidar mapped the floor as
  walls. Frictionless caster, symmetric DiffDrive accel/velocity
  limits, lidar frame set via <ignition_frame_id>.
- spawn_swarm.launch.py: drop the hand-typed lidar static TF, now
  redundant.

Re-test: 0.0 deg tilt on all three robots; SLAM corrections down from
20-44 cm jumps to a few cm.

File: src/swarm_bringup/urdf/rover.urdf.xacro (robot description, xacro)
@@ -28,4 +28,11 @@
   <xacro:property name="lidar_range"   value="${6.0  if is_scout else 12.0}" />
   <xacro:property name="lidar_samples" value="${360  if is_scout else 720}" />
+  <!-- How far the chassis (and the caster and lidar with it) sits ahead of
+       the wheel axle. The robot pivots on the axle, so the center of mass
+       must be clearly ahead of it: at 0 it was only 3-6 mm ahead, and any
+       forward acceleration tipped the rovers onto their tails (measured
+       15.2 deg scout / 12.9 deg mapper). These offsets raise the tip
+       threshold to roughly 4.7 / 6 m/s^2, well above the DiffDrive limit. -->
+  <xacro:property name="chassis_offset_x" value="${0.03 if is_scout else 0.06}" />
   <!-- ===================================================================
        Links
@@ -47,5 +54,5 @@
   <joint name="base_to_chassis" type="fixed">
     <parent link="base_link" /><child link="chassis_link" />
-    <origin xyz="0 0 ${wheel_radius}" rpy="0 0 0" />
+    <origin xyz="${chassis_offset_x} 0 ${wheel_radius}" rpy="0 0 0" />
   </joint>
   <!-- wheels: macro'd so left/right only differ by Y sign -->
@@ -73,5 +80,6 @@
   <xacro:wheel side="left"  y_sign="1" />
   <xacro:wheel side="right" y_sign="-1" />
-  <!-- a simple caster so the chassis doesn't tip -->
+  <!-- front caster at the chassis nose (frictionless: see the gazebo block
+       for caster_link below) -->
   <link name="caster_link">
     <visual><geometry><sphere radius="${wheel_radius * 0.6}" /></geometry></visual>
@@ -84,5 +92,5 @@
   <joint name="caster_joint" type="fixed">
     <parent link="base_link" /><child link="caster_link" />
-    <origin xyz="${chassis_len/2 - wheel_radius*0.6} 0 ${-wheel_radius*0.4}" rpy="0 0 0" />
+    <origin xyz="${chassis_offset_x + chassis_len/2 - wheel_radius*0.6} 0 ${-wheel_radius*0.4}" rpy="0 0 0" />
   </joint>
   <!-- lidar mast -->
@@ -124,5 +132,15 @@
       <wheel_separation>${wheel_sep}</wheel_separation>
       <wheel_radius>${wheel_radius}</wheel_radius>
+      <!-- Symmetric limits: with only max_linear_acceleration set, stops,
+           reverse starts and turns were instantaneous (wheel slip), and the
+           per-class speed caps above were never applied. -->
       <max_linear_acceleration>1.0</max_linear_acceleration>
+      <min_linear_acceleration>-1.0</min_linear_acceleration>
+      <max_angular_acceleration>2.0</max_angular_acceleration>
+      <min_angular_acceleration>-2.0</min_angular_acceleration>
+      <max_linear_velocity>${max_lin_vel}</max_linear_velocity>
+      <min_linear_velocity>${-max_lin_vel}</min_linear_velocity>
+      <max_angular_velocity>${max_ang_vel}</max_angular_velocity>
+      <min_angular_velocity>${-max_ang_vel}</min_angular_velocity>
       <topic>/model/${name}/cmd_vel</topic>
       <odom_topic>/model/${name}/odometry</odom_topic>
@@ -145,5 +163,9 @@
     <sensor name="lidar" type="gpu_lidar">
       <topic>/world/exploration_test/model/${name}/lidar</topic>
-      <frame_id>lidar_link</frame_id>
+      <!-- Fortress ignores plain <frame_id> (scans came out as
+           <name>/base_link/lidar). ignition_frame_id stamps them with the
+           prefixed link robot_state_publisher already publishes, so the
+           scan TF follows this xacro instead of a hand-typed static TF. -->
+      <ignition_frame_id>${name}/lidar_link</ignition_frame_id>
       <update_rate>10</update_rate>
       <always_on>true</always_on>
@@ -165,4 +187,11 @@
     </sensor>
   </gazebo>
+  <!-- Frictionless caster: it now carries real weight, and a mu=1 sphere
+       would drag in turns and corrupt odometry. This reference survives
+       the URDF->SDF fixed-joint lumping into base_link. -->
+  <gazebo reference="caster_link">
+    <mu1>0.0</mu1>
+    <mu2>0.0</mu2>
+  </gazebo>
   <gazebo reference="imu_link">
     <sensor name="imu" type="imu">
